File: LightSensor.sch (KiCad schematic (older format))
At the start: 4 parts, among them U302 VEML7700

Commit message: initial layout
Parts:
- renumbered C302 to C301, R306 to R301, R307 to R302, U302 to U301
Changed lines of the file:
@@
 $EndDescr
 $Comp
-L TMPCB_R2:VEML7700 U302
+L TMPCB_R2:VEML7700 U301
 U 1 1 61A804E2
 P 5550 3550
-F 0 "U302" H 5778 3687 50  0000 L CNN
+F 0 "U301" H 5778 3687 50  0000 L CNN
 F 1 "VEML7700" H 5778 3596 50  0000 L CNN
 F 2 "TMPPCB_R2:SMD4-X07Y16P127" H 5350 3800 50  0001 C CNN
@@
 $EndComp
 $Comp
-L power:+3V3 #PWR0304
+L power:+3V3 #PWR0301
 U 1 1 61A81201
 P 4750 3250
-F 0 "#PWR0304" H 4750 3100 50  0001 C CNN
+F 0 "#PWR0301" H 4750 3100 50  0001 C CNN
 F 1 "+3V3" H 4765 3423 50  0000 C CNN
 F 2 "" H 4750 3250 50  0001 C CNN
@@
 $EndComp
 $Comp
-L power:GND #PWR0305
+L power:GND #PWR0302
 U 1 1 61A81AE1
 P 4750 3950
-F 0 "#PWR0305" H 4750 3700 50  0001 C CNN
+F 0 "#PWR0302" H 4750 3700 50  0001 C CNN
 F 1 "GND" H 4755 3777 50  0000 C CNN
 F 2 "" H 4750 3950 50  0001 C CNN
@@
 $EndComp
 $Comp
-L Device:C_Small C302
+L Device:C_Small C301
 U 1 1 61A8235A
 P 4750 3550
-F 0 "C302" H 4550 3600 50  0000 L CNN
+F 0 "C301" H 4550 3600 50  0000 L CNN
 F 1 "10 uF 10% 10V" H 4400 3500 50  0000 L CNN
 F 2 "Capacitor_SMD:C_0805_2012Metric_Pad1.18x1.45mm_HandSolder" H 4750 3550 50  0001 C CNN
@@
 	5150 3100 5250 3100
 $Comp
-L power:+3V3 #PWR0306
+L power:+3V3 #PWR0303
 U 1 1 61ABAE97
 P 5250 2750
-F 0 "#PWR0306" H 5250 2600 50  0001 C CNN
+F 0 "#PWR0303" H 5250 2600 50  0001 C CNN
 F 1 "+3V3" H 5265 2923 50  0000 C CNN
 F 2 "" H 5250 2750 50  0001 C CNN
@@
 $EndComp
 $Comp
-L Device:R_Small_US R306
+L Device:R_Small_US R301
 U 1 1 61ABB356
 P 5250 2850
-F 0 "R306" H 5318 2896 50  0000 L CNN
+F 0 "R301" H 5318 2896 50  0000 L CNN
 F 1 "4.7k 5%" H 5318 2805 50  0000 L CNN
 F 2 "Resistor_SMD:R_0805_2012Metric_Pad1.20x1.40mm_HandSolder" H 5250 2850 50  0001 C CNN
@@
 	5250 3100 5350 3100
 $Comp
-L power:+3V3 #PWR0307
+L power:+3V3 #PWR0304
 U 1 1 61ABE8BA
 P 5500 4100
-F 0 "#PWR0307" H 5500 3950 50  0001 C CNN
+F 0 "#PWR0304" H 5500 3950 50  0001 C CNN
 F 1 "+3V3" H 5515 4273 50  0000 C CNN
 F 2 "" H 5500 4100 50  0001 C CNN
@@
 $EndComp
 $Comp
-L Device:R_Small_US R307
+L Device:R_Small_US R302
 U 1 1 61ABE8C0
 P 5500 4200
-F 0 "R307" H 5568 4246 50  0000 L CNN
+F 0 "R302" H 5568 4246 50  0000 L CNN
 F 1 "4.7k 5%" H 5568 4155 50  0000 L CNN
 F 2 "Resistor_SMD:R_0805_2012Metric_Pad1.20x1.40mm_HandSolder" H 5500 4200 50  0001 C CNN

Commit message: Fix design error in PI4ULS5V201TAEX. Reset and reassigned all annotations.
Parts:
- renumbered C301 to C201, R301 to R201, R302 to R202, U301 to U201
Changed lines of the file:
@@
 $EndDescr
 $Comp
-L TMPCB_R2:VEML7700 U301
+L TMPCB_R2:VEML7700 U201
 U 1 1 61A804E2
 P 5550 3550
-F 0 "U301" H 5778 3687 50  0000 L CNN
+F 0 "U201" H 5778 3687 50  0000 L CNN
 F 1 "VEML7700" H 5778 3596 50  0000 L CNN
 F 2 "TMPPCB_R2:SMD4-X07Y16P127" H 5350 3800 50  0001 C CNN
@@
 $EndComp
 $Comp
-L power:+3V3 #PWR0301
+L power:+3V3 #PWR0201
 U 1 1 61A81201
 P 4750 3250
-F 0 "#PWR0301" H 4750 3100 50  0001 C CNN
+F 0 "#PWR0201" H 4750 3100 50  0001 C CNN
 F 1 "+3V3" H 4765 3423 50  0000 C CNN
 F 2 "" H 4750 3250 50  0001 C CNN
@@
 $EndComp
 $Comp
-L power:GND #PWR0302
+L power:GND #PWR0202
 U 1 1 61A81AE1
 P 4750 3950
-F 0 "#PWR0302" H 4750 3700 50  0001 C CNN
+F 0 "#PWR0202" H 4750 3700 50  0001 C CNN
 F 1 "GND" H 4755 3777 50  0000 C CNN
 F 2 "" H 4750 3950 50  0001 C CNN
@@
 $EndComp
 $Comp
-L Device:C_Small C301
+L Device:C_Small C201
 U 1 1 61A8235A
 P 4750 3550
-F 0 "C301" H 4550 3600 50  0000 L CNN
+F 0 "C201" H 4550 3600 50  0000 L CNN
 F 1 "10 uF 10% 10V" H 4400 3500 50  0000 L CNN
 F 2 "Capacitor_SMD:C_0805_2012Metric_Pad1.18x1.45mm_HandSolder" H 4750 3550 50  0001 C CNN
@@
 	5150 3100 5250 3100
 $Comp
-L power:+3V3 #PWR0303
+L power:+3V3 #PWR0203
 U 1 1 61ABAE97
 P 5250 2750
-F 0 "#PWR0303" H 5250 2600 50  0001 C CNN
+F 0 "#PWR0203" H 5250 2600 50  0001 C CNN
 F 1 "+3V3" H 5265 2923 50  0000 C CNN
 F 2 "" H 5250 2750 50  0001 C CNN
@@
 $EndComp
 $Comp
-L Device:R_Small_US R301
+L Device:R_Small_US R201
 U 1 1 61ABB356
 P 5250 2850
-F 0 "R301" H 5318 2896 50  0000 L CNN
+F 0 "R201" H 5318 2896 50  0000 L CNN
 F 1 "4.7k 5%" H 5318 2805 50  0000 L CNN
 F 2 "Resistor_SMD:R_0805_2012Metric_Pad1.20x1.40mm_HandSolder" H 5250 2850 50  0001 C CNN
@@
 	5250 3100 5350 3100
 $Comp
-L power:+3V3 #PWR0304
+L power:+3V3 #PWR0204
 U 1 1 61ABE8BA
 P 5500 4100
-F 0 "#PWR0304" H 5500 3950 50  0001 C CNN
+F 0 "#PWR0204" H 5500 3950 50  0001 C CNN
 F 1 "+3V3" H 5515 4273 50  0000 C CNN
 F 2 "" H 5500 4100 50  0001 C CNN
@@
 $EndComp
 $Comp
-L Device:R_Small_US R302
+L Device:R_Small_US R202
 U 1 1 61ABE8C0
 P 5500 4200
-F 0 "R302" H 5568 4246 50  0000 L CNN
+F 0 "R202" H 5568 4246 50  0000 L CNN
 F 1 "4.7k 5%" H 5568 4155 50  0000 L CNN
 F 2 "Resistor_SMD:R_0805_2012Metric_Pad1.20x1.40mm_HandSolder" H 5500 4200 50  0001 C CNN
