File: RGBDrvier.sch (KiCad schematic (older format))
At the start: 7 parts, among them U301 NLSF595

Commit message: Added PCA9745B16B. Updated schematic. ERC Passes.
Parts:
- removed U301: NLSF595, Package_SO:TSSOP-16_4.4x5mm_P0.65mm, symbol TMPCB_R2:NLSF595
- added R2701: 1k 5%, Resistor_SMD:R_0805_2012Metric_Pad1.20x1.40mm_HandSolder, symbol Device:R_Small_US
- added R2702: 100k 5%, Resistor_SMD:R_0805_2012Metric_Pad1.20x1.40mm_HandSolder, symbol Device:R_Small_US
- added U2701: PCA9745BTWJ, HTSSOP28_4P5X9P8_NXP, symbol Macro_Keyboard:PCA9745BTWJ
Connections:
- net labels added: DRIVER_LED_B_5V, DRIVER_LED_CS_3V3, DRIVER_LED_G_5V, DRIVER_LED_R_5V, SPI_MISO_3V
- net labels removed: DRIVER_LED_B, DRIVER_LED_G, DRIVER_LED_R, DRIVER_LED_RCK, NOT_OE, NOT_SCLR, RCK, SCK, SI, VCC
- no-connect marks 6 -> 13
Other:
- moved on the sheet: C301, R301, R302, R303, R304, R305

Commit message: initial layout
Parts:
- U2701: footprint HTSSOP28_4P5X9P8_NXP -> Macro Keyboard:PCA9745BTWJ
- renumbered C301 to C2701, R301 to R2701, R305 to R2702, R2701 to R2703, R304 to R2704, R2702 to R2705, R302 to R2706, R303 to R2707
Changed lines of the file:
@@
 $EndDescr
 $Comp
-L Device:R_Small_US R304
+L Device:R_Small_US R2704
 U 1 1 61A3FADF
 P 4450 3300
-F 0 "R304" V 4550 3300 50  0000 C CNN
+F 0 "R2704" V 4550 3300 50  0000 C CNN
 F 1 "1k 5%" V 4350 3300 50  0000 C CNN
 F 2 "Resistor_SMD:R_0805_2012Metric_Pad1.20x1.40mm_HandSolder" H 4450 3300 50  0001 C CNN
@@
 $EndComp
 $Comp
-L Device:R_Small_US R305
+L Device:R_Small_US R2702
 U 1 1 61A41C08
 P 4250 4150
-F 0 "R305" V 4350 4150 50  0000 C CNN
+F 0 "R2702" V 4350 4150 50  0000 C CNN
 F 1 "1k 5%" V 4150 4150 50  0000 C CNN
 F 2 "Resistor_SMD:R_0805_2012Metric_Pad1.20x1.40mm_HandSolder" H 4250 4150 50  0001 C CNN
@@
 $EndComp
 $Comp
-L Device:R_Small_US R303
+L Device:R_Small_US R2707
 U 1 1 61A429FE
 P 7650 3350
-F 0 "R303" V 7550 3350 50  0000 C CNN
+F 0 "R2707" V 7550 3350 50  0000 C CNN
 F 1 "1k 5%" V 7750 3350 50  0000 C CNN
 F 2 "Resistor_SMD:R_0805_2012Metric_Pad1.20x1.40mm_HandSolder" H 7650 3350 50  0001 C CNN
@@
 $EndComp
 $Comp
-L Device:R_Small_US R301
+L Device:R_Small_US R2701
 U 1 1 61A3D9CE
 P 4050 3750
-F 0 "R301" V 4150 3750 50  0000 C CNN
+F 0 "R2701" V 4150 3750 50  0000 C CNN
 F 1 "4.7k 5%" V 3950 3750 50  0000 C CNN
 F 2 "Resistor_SMD:R_0805_2012Metric_Pad1.20x1.40mm_HandSolder" H 4050 3750 50  0001 C CNN
@@
 $EndComp
 $Comp
-L Device:C_Small C301
+L Device:C_Small C2701
 U 1 1 61A3C95F
 P 6800 2550
-F 0 "C301" H 6708 2504 50  0000 R CNN
+F 0 "C2701" H 6708 2504 50  0000 R CNN
 F 1 "1 uF 10% 10V" V 6900 2800 50  0000 R CNN
 F 2 "Capacitor_SMD:C_0805_2012Metric_Pad1.18x1.45mm_HandSolder" H 6800 2550 50  0001 C CNN
@@
 DRIVER_LED_B_5V
 $Comp
-L Device:R_Small_US R302
+L Device:R_Small_US R2706
 U 1 1 61A5BA43
 P 7650 2950
-F 0 "R302" V 7550 2950 50  0000 C CNN
+F 0 "R2706" V 7550 2950 50  0000 C CNN
 F 1 "1k 5%" V 7750 2950 50  0000 C CNN
 F 2 "Resistor_SMD:R_0805_2012Metric_Pad1.20x1.40mm_HandSolder" H 7650 2950 50  0001 C CNN
@@
 SPI_MOSI_3V
 $Comp
-L power:GND #PWR0301
+L power:GND #PWR02701
 U 1 1 61A5E7D1
 P 4050 3850
-F 0 "#PWR0301" H 4050 3600 50  0001 C CNN
+F 0 "#PWR02701" H 4050 3600 50  0001 C CNN
 F 1 "GND" H 4055 3677 50  0000 C CNN
 F 2 "" H 4050 3850 50  0001 C CNN
@@
 DRIVER_LED_CS_3V3
 $Comp
-L power:+3V3 #PWR0101
+L power:+3V3 #PWR02706
 U 1 1 61A270A5
 P 6800 2300
-F 0 "#PWR0101" H 6800 2150 50  0001 C CNN
+F 0 "#PWR02706" H 6800 2150 50  0001 C CNN
 F 1 "+3V3" H 6815 2473 50  0000 C CNN
 F 2 "" H 6800 2300 50  0001 C CNN
@@
 	6800 2450 6800 2400
 $Comp
-L power:GND #PWR0102
+L power:GND #PWR02707
 U 1 1 61A29573
 P 6800 2650
-F 0 "#PWR0102" H 6800 2400 50  0001 C CNN
+F 0 "#PWR02707" H 6800 2400 50  0001 C CNN
 F 1 "GND" H 6805 2477 50  0000 C CNN
 F 2 "" H 6800 2650 50  0001 C CNN
@@
 $EndComp
 $Comp
-L power:GND #PWR0103
+L power:GND #PWR02708
 U 1 1 61A29979
 P 6850 3200
-F 0 "#PWR0103" H 6850 2950 50  0001 C CNN
+F 0 "#PWR02708" H 6850 2950 50  0001 C CNN
 F 1 "GND" H 6855 3027 50  0000 C CNN
 F 2 "" H 6850 3200 50  0001 C CNN
@@
 $EndComp
 $Comp
-L power:GND #PWR0104
+L power:GND #PWR02709
 U 1 1 61A29FBA
 P 6850 3700
-F 0 "#PWR0104" H 6850 3450 50  0001 C CNN
+F 0 "#PWR02709" H 6850 3450 50  0001 C CNN
 F 1 "GND" H 6855 3527 50  0000 C CNN
 F 2 "" H 6850 3700 50  0001 C CNN
@@
 $EndComp
 $Comp
-L power:GND #PWR0105
+L power:GND #PWR02710
 U 1 1 61A2A2ED
 P 6850 4200
-F 0 "#PWR0105" H 6850 3950 50  0001 C CNN
+F 0 "#PWR02710" H 6850 3950 50  0001 C CNN
 F 1 "GND" H 6855 4027 50  0000 C CNN
 F 2 "" H 6850 4200 50  0001 C CNN
@@
 $EndComp
 $Comp
-L power:GND #PWR0106
+L power:GND #PWR02704
 U 1 1 61A2AAFC
 P 5050 3300
-F 0 "#PWR0106" H 5050 3050 50  0001 C CNN
+F 0 "#PWR02704" H 5050 3050 50  0001 C CNN
 F 1 "GND" H 5055 3127 50  0000 C CNN
 F 2 "" H 5050 3300 50  0001 C CNN
@@
 $EndComp
 $Comp
-L power:GND #PWR0107
+L power:GND #PWR02705
 U 1 1 61A2B14E
 P 5050 4100
-F 0 "#PWR0107" H 5050 3850 50  0001 C CNN
+F 0 "#PWR02705" H 5050 3850 50  0001 C CNN
 F 1 "GND" H 5055 3927 50  0000 C CNN
 F 2 "" H 5050 4100 50  0001 C CNN
@@
 	4700 3300 4700 3400
 $Comp
-L Device:R_Small_US R2701
+L Device:R_Small_US R2703
 U 1 1 61A47F87
 P 4450 2900
-F 0 "R2701" V 4350 2900 50  0000 C CNN
+F 0 "R2703" V 4350 2900 50  0000 C CNN
 F 1 "1k 5%" V 4550 2900 50  0000 C CNN
 F 2 "Resistor_SMD:R_0805_2012Metric_Pad1.20x1.40mm_HandSolder" H 4450 2900 50  0001 C CNN
@@
 	4750 2900 4550 2900
 $Comp
-L power:GND #PWR0108
+L power:GND #PWR02703
 U 1 1 61A495AF
 P 4350 2900
-F 0 "#PWR0108" H 4350 2650 50  0001 C CNN
+F 0 "#PWR02703" H 4350 2650 50  0001 C CNN
 F 1 "GND" H 4355 2727 50  0000 C CNN
 F 2 "" H 4350 2900 50  0001 C CNN
@@
 $EndComp
 $Comp
-L power:GND #PWR0109
+L power:GND #PWR02702
 U 1 1 61A4BA00
 P 4250 4250
-F 0 "#PWR0109" H 4250 4000 50  0001 C CNN
+F 0 "#PWR02702" H 4250 4000 50  0001 C CNN
 F 1 "GND" H 4255 4077 50  0000 C CNN
 F 2 "" H 4250 4250 50  0001 C CNN
@@
 $EndComp
 $Comp
-L Device:R_Small_US R2702
+L Device:R_Small_US R2705
 U 1 1 61A57FAE
 P 7600 3850
-F 0 "R2702" V 7500 3850 50  0000 C CNN
+F 0 "R2705" V 7500 3850 50  0000 C CNN
 F 1 "100k 5%" V 7700 3850 50  0000 C CNN
 F 2 "Resistor_SMD:R_0805_2012Metric_Pad1.20x1.40mm_HandSolder" H 7600 3850 50  0001 C CNN
@@
 $EndComp
 $Comp
-L power:+3V3 #PWR0110
+L power:+3V3 #PWR02711
 U 1 1 61A58237
 P 7900 3800
-F 0 "#PWR0110" H 7900 3650 50  0001 C CNN
+F 0 "#PWR02711" H 7900 3650 50  0001 C CNN
 F 1 "+3V3" H 7915 3973 50  0000 C CNN
 F 2 "" H 7900 3800 50  0001 C CNN
@@
 F 0 "U2701" H 5950 3587 60  0000 C CNN
 F 1 "PCA9745BTWJ" H 5950 3481 60  0000 C CNN
-F 2 "HTSSOP28_4P5X9P8_NXP" H 5950 3440 60  0001 C CNN
+F 2 "Macro Keyboard:PCA9745BTWJ" H 5950 3440 60  0001 C CNN
 F 3 "" H 5050 3200 60  0000 C CNN
 	1    5050 3200
 	1    0    0    -1
 $EndComp
-Connection ~ 6850 4200
-Connection ~ 6850 3700
-Connection ~ 6850 3600
-Connection ~ 6850 3500
-Connection ~ 6850 3400
-Connection ~ 6850 3300
-Connection ~ 6850 3200
 Wire Wire Line
 	4750 3200 5050 3200

Commit message: Layout completed. Design check passes.
Connections:
- net DRIVER_LED_SW2_R_5V: now reaches U2701.11 (LED4)
- net DRIVER_LED_SW2_G_5V: now reaches U2701.12 (LED5)
- net DRIVER_LED_SW2_B_5V: now reaches U2701.13 (LED6)
- net DRIVER_LED_B_5V renamed DRIVER_LED_SW1_B_5V
- net DRIVER_LED_G_5V renamed DRIVER_LED_SW1_G_5V
- net DRIVER_LED_R_5V renamed DRIVER_LED_SW1_R_5V
- no-connect marks 13 -> 10
Changed lines of the file:
@@
 $Descr A4 11693 8268
 encoding utf-8
-Sheet 27 30
+Sheet 26 30
 Title ""
 Date ""
@@
 $EndComp
 Text HLabel 5050 3700 0    50   Input ~ 0
-DRIVER_LED_R_5V
+DRIVER_LED_SW1_R_5V
 Text HLabel 5050 3800 0    50   Input ~ 0
-DRIVER_LED_G_5V
+DRIVER_LED_SW1_G_5V
 Text HLabel 5050 3900 0    50   Input ~ 0
-DRIVER_LED_B_5V
+DRIVER_LED_SW1_B_5V
 $Comp
 L Device:R_Small_US R2706
@@
 NoConn ~ 6850 4600
 NoConn ~ 5050 4000
-NoConn ~ 5050 4200
-NoConn ~ 5050 4300
-NoConn ~ 5050 4400
 NoConn ~ 5050 4500
 Text GLabel 4200 3300 0    50   Input ~ 0
@@
 Wire Wire Line
 	4250 3600 5050 3600
+Text HLabel 5050 4400 0    50   Input ~ 0
+DRIVER_LED_SW2_B_5V
+Text HLabel 5050 4300 0    50   Input ~ 0
+DRIVER_LED_SW2_G_5V
+Text HLabel 5050 4200 0    50   Input ~ 0
+DRIVER_LED_SW2_R_5V
 $EndSCHEMATC

Commit message: Checkpoint
Parts:
- R2705: Digikey PN RMCF0805JT1K00CT-ND -> RMCF0805JT100KCT-ND; MFG # RMCF0805JT1K00 -> RMCF0805JT100K
- U2701: Digikey PN (none) -> 568-14156-1-ND; MFG (none) -> NXP USA Inc.; MFG # (none) -> PCA9745BTWJ
Changed lines of the file:
@@
 F 2 "Resistor_SMD:R_0805_2012Metric_Pad1.20x1.40mm_HandSolder" H 7600 3850 50  0001 C CNN
 F 3 "https://www.seielect.com/catalog/sei-rmcf_rmcp.pdf" H 7600 3850 50  0001 C CNN
-F 4 "RMCF0805JT1K00CT-ND" H 7600 3850 50  0001 C CNN "Digikey PN"
+F 4 "RMCF0805JT100KCT-ND" H 7600 3850 50  0001 C CNN "Digikey PN"
 F 5 "Stackpole Electronics Inc" H 7600 3850 50  0001 C CNN "MFG"
-F 6 "RMCF0805JT1K00" H 7600 3850 50  0001 C CNN "MFG #"
+F 6 "RMCF0805JT100K" H 7600 3850 50  0001 C CNN "MFG #"
 	1    7600 3850
 	0    1    1    0
@@
 F 1 "PCA9745BTWJ" H 5950 3481 60  0000 C CNN
 F 2 "Macro Keyboard:PCA9745BTWJ" H 5950 3440 60  0001 C CNN
-F 3 "" H 5050 3200 60  0000 C CNN
+F 3 "https://www.nxp.com/docs/en/data-sheet/PCA9745B.pdf" H 5050 3200 60  0000 C CNN
+F 4 "568-14156-1-ND" H 5050 3200 50  0001 C CNN "Digikey PN"
+F 5 "NXP USA Inc." H 5050 3200 50  0001 C CNN "MFG"
+F 6 "PCA9745BTWJ" H 5050 3200 50  0001 C CNN "MFG #"
 	1    5050 3200
 	1    0    0    -1

Commit message: Fix design error in PI4ULS5V201TAEX. Reset and reassigned all annotations.
Parts:
- renumbered C2701 to C2601, R2701 to R2601, R2702 to R2602, R2703 to R2603, R2704 to R2604, R2705 to R2605, R2706 to R2606, R2707 to R2607, U2701 to U2601
Changed lines of the file:
@@
 $EndDescr
 $Comp
-L Device:R_Small_US R2704
+L Device:R_Small_US R2604
 U 1 1 61A3FADF
 P 4450 3300
-F 0 "R2704" V 4550 3300 50  0000 C CNN
+F 0 "R2604" V 4550 3300 50  0000 C CNN
 F 1 "1k 5%" V 4350 3300 50  0000 C CNN
 F 2 "Resistor_SMD:R_0805_2012Metric_Pad1.20x1.40mm_HandSolder" H 4450 3300 50  0001 C CNN
@@
 $EndComp
 $Comp
-L Device:R_Small_US R2702
+L Device:R_Small_US R2602
 U 1 1 61A41C08
 P 4250 4150
-F 0 "R2702" V 4350 4150 50  0000 C CNN
+F 0 "R2602" V 4350 4150 50  0000 C CNN
 F 1 "1k 5%" V 4150 4150 50  0000 C CNN
 F 2 "Resistor_SMD:R_0805_2012Metric_Pad1.20x1.40mm_HandSolder" H 4250 4150 50  0001 C CNN
@@
 $EndComp
 $Comp
-L Device:R_Small_US R2707
+L Device:R_Small_US R2607
 U 1 1 61A429FE
 P 7650 3350
-F 0 "R2707" V 7550 3350 50  0000 C CNN
+F 0 "R2607" V 7550 3350 50  0000 C CNN
 F 1 "1k 5%" V 7750 3350 50  0000 C CNN
 F 2 "Resistor_SMD:R_0805_2012Metric_Pad1.20x1.40mm_HandSolder" H 7650 3350 50  0001 C CNN
@@
 $EndComp
 $Comp
-L Device:R_Small_US R2701
+L Device:R_Small_US R2601
 U 1 1 61A3D9CE
 P 4050 3750
-F 0 "R2701" V 4150 3750 50  0000 C CNN
+F 0 "R2601" V 4150 3750 50  0000 C CNN
 F 1 "4.7k 5%" V 3950 3750 50  0000 C CNN
 F 2 "Resistor_SMD:R_0805_2012Metric_Pad1.20x1.40mm_HandSolder" H 4050 3750 50  0001 C CNN
@@
 $EndComp
 $Comp
-L Device:C_Small C2701
+L Device:C_Small C2601
 U 1 1 61A3C95F
 P 6800 2550
-F 0 "C2701" H 6708 2504 50  0000 R CNN
+F 0 "C2601" H 6708 2504 50  0000 R CNN
 F 1 "1 uF 10% 10V" V 6900 2800 50  0000 R CNN
 F 2 "Capacitor_SMD:C_0805_2012Metric_Pad1.18x1.45mm_HandSolder" H 6800 2550 50  0001 C CNN
@@
 DRIVER_LED_SW1_B_5V
 $Comp
-L Device:R_Small_US R2706
+L Device:R_Small_US R2606
 U 1 1 61A5BA43
 P 7650 2950
-F 0 "R2706" V 7550 2950 50  0000 C CNN
+F 0 "R2606" V 7550 2950 50  0000 C CNN
 F 1 "1k 5%" V 7750 2950 50  0000 C CNN
 F 2 "Resistor_SMD:R_0805_2012Metric_Pad1.20x1.40mm_HandSolder" H 7650 2950 50  0001 C CNN
@@
 SPI_MOSI_3V
 $Comp
-L power:GND #PWR02701
+L power:GND #PWR02601
 U 1 1 61A5E7D1
 P 4050 3850
-F 0 "#PWR02701" H 4050 3600 50  0001 C CNN
+F 0 "#PWR02601" H 4050 3600 50  0001 C CNN
 F 1 "GND" H 4055 3677 50  0000 C CNN
 F 2 "" H 4050 3850 50  0001 C CNN
@@
 DRIVER_LED_CS_3V3
 $Comp
-L power:+3V3 #PWR02706
+L power:+3V3 #PWR02606
 U 1 1 61A270A5
 P 6800 2300
-F 0 "#PWR02706" H 6800 2150 50  0001 C CNN
+F 0 "#PWR02606" H 6800 2150 50  0001 C CNN
 F 1 "+3V3" H 6815 2473 50  0000 C CNN
 F 2 "" H 6800 2300 50  0001 C CNN
@@
 	6800 2450 6800 2400
 $Comp
-L power:GND #PWR02707
+L power:GND #PWR02607
 U 1 1 61A29573
 P 6800 2650
-F 0 "#PWR02707" H 6800 2400 50  0001 C CNN
+F 0 "#PWR02607" H 6800 2400 50  0001 C CNN
 F 1 "GND" H 6805 2477 50  0000 C CNN
 F 2 "" H 6800 2650 50  0001 C CNN
@@
 $EndComp
 $Comp
-L power:GND #PWR02708
+L power:GND #PWR02608
 U 1 1 61A29979
 P 6850 3200
-F 0 "#PWR02708" H 6850 2950 50  0001 C CNN
+F 0 "#PWR02608" H 6850 2950 50  0001 C CNN
 F 1 "GND" H 6855 3027 50  0000 C CNN
 F 2 "" H 6850 3200 50  0001 C CNN
@@
 $EndComp
 $Comp
-L power:GND #PWR02709
+L power:GND #PWR02609
 U 1 1 61A29FBA
 P 6850 3700
-F 0 "#PWR02709" H 6850 3450 50  0001 C CNN
+F 0 "#PWR02609" H 6850 3450 50  0001 C CNN
 F 1 "GND" H 6855 3527 50  0000 C CNN
 F 2 "" H 6850 3700 50  0001 C CNN
@@
 $EndComp
 $Comp
-L power:GND #PWR02710
+L power:GND #PWR02610
 U 1 1 61A2A2ED
 P 6850 4200
-F 0 "#PWR02710" H 6850 3950 50  0001 C CNN
+F 0 "#PWR02610" H 6850 3950 50  0001 C CNN
 F 1 "GND" H 6855 4027 50  0000 C CNN
 F 2 "" H 6850 4200 50  0001 C CNN
@@
 $EndComp
 $Comp
-L power:GND #PWR02704
+L power:GND #PWR02604
 U 1 1 61A2AAFC
 P 5050 3300
-F 0 "#PWR02704" H 5050 3050 50  0001 C CNN
+F 0 "#PWR02604" H 5050 3050 50  0001 C CNN
 F 1 "GND" H 5055 3127 50  0000 C CNN
 F 2 "" H 5050 3300 50  0001 C CNN
@@
 $EndComp
 $Comp
-L power:GND #PWR02705
+L power:GND #PWR02605
 U 1 1 61A2B14E
 P 5050 4100
-F 0 "#PWR02705" H 5050 3850 50  0001 C CNN
+F 0 "#PWR02605" H 5050 3850 50  0001 C CNN
 F 1 "GND" H 5055 3927 50  0000 C CNN
 F 2 "" H 5050 4100 50  0001 C CNN
@@
 	4700 3300 4700 3400
 $Comp
-L Device:R_Small_US R2703
+L Device:R_Small_US R2603
 U 1 1 61A47F87
 P 4450 2900
-F 0 "R2703" V 4350 2900 50  0000 C CNN
+F 0 "R2603" V 4350 2900 50  0000 C CNN
 F 1 "1k 5%" V 4550 2900 50  0000 C CNN
 F 2 "Resistor_SMD:R_0805_2012Metric_Pad1.20x1.40mm_HandSolder" H 4450 2900 50  0001 C CNN
@@
 	4750 2900 4550 2900
 $Comp
-L power:GND #PWR02703
+L power:GND #PWR02603
 U 1 1 61A495AF
 P 4350 2900
-F 0 "#PWR02703" H 4350 2650 50  0001 C CNN
+F 0 "#PWR02603" H 4350 2650 50  0001 C CNN
 F 1 "GND" H 4355 2727 50  0000 C CNN
 F 2 "" H 4350 2900 50  0001 C CNN
@@
 $EndComp
 $Comp
-L power:GND #PWR02702
+L power:GND #PWR02602
 U 1 1 61A4BA00
 P 4250 4250
-F 0 "#PWR02702" H 4250 4000 50  0001 C CNN
+F 0 "#PWR02602" H 4250 4000 50  0001 C CNN
 F 1 "GND" H 4255 4077 50  0000 C CNN
 F 2 "" H 4250 4250 50  0001 C CNN
@@
 $EndComp
 $Comp
-L Device:R_Small_US R2705
+L Device:R_Small_US R2605
 U 1 1 61A57FAE
 P 7600 3850
-F 0 "R2705" V 7500 3850 50  0000 C CNN
+F 0 "R2605" V 7500 3850 50  0000 C CNN
 F 1 "100k 5%" V 7700 3850 50  0000 C CNN
 F 2 "Resistor_SMD:R_0805_2012Metric_Pad1.20x1.40mm_HandSolder" H 7600 3850 50  0001 C CNN
@@
 $EndComp
 $Comp
-L power:+3V3 #PWR02711
+L power:+3V3 #PWR02611
 U 1 1 61A58237
 P 7900 3800
-F 0 "#PWR02711" H 7900 3650 50  0001 C CNN
+F 0 "#PWR02611" H 7900 3650 50  0001 C CNN
 F 1 "+3V3" H 7915 3973 50  0000 C CNN
 F 2 "" H 7900 3800 50  0001 C CNN
@@
 	4250 4050 4250 3600
 $Comp
-L Macro_Keyboard:PCA9745BTWJ U2701
+L Macro_Keyboard:PCA9745BTWJ U2601
 U 1 1 61A3EABF
 P 5050 3200
-F 0 "U2701" H 5950 3587 60  0000 C CNN
+F 0 "U2601" H 5950 3587 60  0000 C CNN
 F 1 "PCA9745BTWJ" H 5950 3481 60  0000 C CNN
 F 2 "Macro Keyboard:PCA9745BTWJ" H 5950 3440 60  0001 C CNN
