File: RotaryEncoder.sch (KiCad schematic (older format))
At the start: 13 parts

Commit message: Added PCA9745B16B. Updated schematic. ERC Passes.
Connections:
- net REnc_LED_B renamed REnc_LED_B_5V
- net REnc_LED_G renamed REnc_LED_G_5V
- net REnc_LED_R renamed REnc_LED_R_5V
Changed lines of the file:
@@
 $EndComp
 Text HLabel 6250 3600 2    50   Output ~ 0
-REnc_LED_R
+REnc_LED_R_5V
 Text HLabel 7100 3700 2    50   Output ~ 0
-REnc_LED_G
+REnc_LED_G_5V
 Text HLabel 8000 3800 2    50   Output ~ 0
-REnc_LED_B
+REnc_LED_B_5V
 Wire Wire Line
 	6900 3700 6050 3700
@@
 	5950 4800 5950 5100
 Wire Wire Line
-	5950 5100 6400 5100
-Wire Wire Line
-	6400 5100 6400 4800
+	5950 5100 6200 5100
 $Comp
 L power:GND #PWR0205
 U 1 1 61A367C9
-P 6400 5100
-F 0 "#PWR0205" H 6400 4850 50  0001 C CNN
-F 1 "GND" H 6405 4927 50  0000 C CNN
-F 2 "" H 6400 5100 50  0001 C CNN
-F 3 "" H 6400 5100 50  0001 C CNN
-	1    6400 5100
+P 6200 5200
+F 0 "#PWR0205" H 6200 4950 50  0001 C CNN
+F 1 "GND" H 6205 5027 50  0000 C CNN
+F 2 "" H 6200 5200 50  0001 C CNN
+F 3 "" H 6200 5200 50  0001 C CNN
+	1    6200 5200
 	1    0    0    -1
 $EndComp
-Connection ~ 6400 5100
 Text HLabel 5650 4550 0    50   Output ~ 0
 REnc_SW
@@
 Wire Wire Line
 	5950 4550 5950 4450
+Connection ~ 6200 5100
+Wire Wire Line
+	6200 5100 6400 5100
+Wire Wire Line
+	6400 5100 6400 4800
+Wire Wire Line
+	6200 5100 6200 5200
 $EndSCHEMATC

Commit message: Layout completed. Design check passes.
Connections:
- net RES_DR: now reaches R205.2, S201.1 (-R)
- net RES_DG: now reaches R208.2, S201.2 (-G)
- net RE_SW_RES: now reaches R206.2, S201.3 (SW)
- net RES_DB: now reaches R209.2, S201.4 (-B)
- net RE_SW_A: now reaches R201.2, R202.1, S201.A
- net RE_SW_B: now reaches R203.2, R204.1, S201.B
Other:
- moved on the sheet: R3005, R3008, R3009
Changed lines of the file:
@@
 $Descr A4 11693 8268
 encoding utf-8
-Sheet 2 30
+Sheet 30 30
 Title ""
 Date ""
@@
 AR Path="/61A047C3/61A23094" Ref="#PWR0203"  Part="1"
 AR Path="/61A55BF3/61A23094" Ref="#PWR0101"  Part="1"
-F 0 "#PWR0101" H 4700 3350 50  0001 C CNN
+F 0 "#PWR0203" H 4700 3350 50  0001 C CNN
 F 1 "GND" H 4600 3600 50  0000 C CNN
 F 2 "" H 4700 3600 50  0001 C CNN
@@
 AR Path="/61A047C3/61A247A0" Ref="#PWR0202"  Part="1"
 AR Path="/61A55BF3/61A247A0" Ref="#PWR0102"  Part="1"
-F 0 "#PWR0102" H 3950 2700 50  0001 C CNN
+F 0 "#PWR0202" H 3950 2700 50  0001 C CNN
 F 1 "+3V3" H 3965 3023 50  0000 C CNN
 F 2 "" H 3950 2850 50  0001 C CNN
@@
 AR Path="/61A047C3/61A24F25" Ref="R202"  Part="1"
 AR Path="/61A55BF3/61A24F25" Ref="R3002"  Part="1"
-F 0 "R202" H 4000 2950 50  0000 R CNN
+F 0 "R3002" H 4000 2950 50  0000 R CNN
 F 1 "47k 5%" H 4150 3050 50  0000 R CNN
 F 2 "Resistor_SMD:R_0805_2012Metric_Pad1.20x1.40mm_HandSolder" H 3800 3000 50  0001 C CNN
@@
 AR Path="/61A047C3/61A25788" Ref="R204"  Part="1"
 AR Path="/61A55BF3/61A25788" Ref="R3004"  Part="1"
-F 0 "R204" H 4032 2954 50  0000 R CNN
+F 0 "R3004" H 4032 2954 50  0000 R CNN
 F 1 "47k 5%" H 4032 3045 50  0000 R CNN
 F 2 "Resistor_SMD:R_0805_2012Metric_Pad1.20x1.40mm_HandSolder" H 4100 3000 50  0001 C CNN
@@
 AR Path="/61A047C3/61A260B2" Ref="R201"  Part="1"
 AR Path="/61A55BF3/61A260B2" Ref="R3001"  Part="1"
-F 0 "R201" V 3700 3450 50  0000 R CNN
+F 0 "R3001" V 3700 3450 50  0000 R CNN
 F 1 "4.7k 5%" V 3500 3550 50  0000 R CNN
 F 2 "Resistor_SMD:R_0805_2012Metric_Pad1.20x1.40mm_HandSolder" H 3600 3400 50  0001 C CNN
@@
 AR Path="/61A047C3/61A2753E" Ref="R203"  Part="1"
 AR Path="/61A55BF3/61A2753E" Ref="R3003"  Part="1"
-F 0 "R203" V 3900 3850 50  0000 R CNN
+F 0 "R3003" V 3900 3850 50  0000 R CNN
 F 1 "4.7k 5%" V 3700 3950 50  0000 R CNN
 F 2 "Resistor_SMD:R_0805_2012Metric_Pad1.20x1.40mm_HandSolder" H 3800 3800 50  0001 C CNN
@@
 AR Path="/61A047C3/61A2842D" Ref="C201"  Part="1"
 AR Path="/61A55BF3/61A2842D" Ref="C3001"  Part="1"
-F 0 "C201" V 3050 4050 50  0000 L CNN
+F 0 "C3001" V 3050 4050 50  0000 L CNN
 F 1 "1 uF 10% 10V" V 3200 3950 50  0000 L CNN
 F 2 "Capacitor_SMD:C_0805_2012Metric_Pad1.18x1.45mm_HandSolder" H 3300 4100 50  0001 C CNN
@@
 AR Path="/61A047C3/61A29140" Ref="C202"  Part="1"
 AR Path="/61A55BF3/61A29140" Ref="C3002"  Part="1"
-F 0 "C202" V 3250 4050 50  0000 L CNN
+F 0 "C3002" V 3250 4050 50  0000 L CNN
 F 1 "1 uF 10% 10V" V 3400 3950 50  0000 L CNN
 F 2 "Capacitor_SMD:C_0805_2012Metric_Pad1.18x1.45mm_HandSolder" H 3500 4100 50  0001 C CNN
@@
 AR Path="/61A047C3/61A2A062" Ref="#PWR0201"  Part="1"
 AR Path="/61A55BF3/61A2A062" Ref="#PWR0103"  Part="1"
-F 0 "#PWR0103" H 3400 4150 50  0001 C CNN
+F 0 "#PWR0201" H 3400 4150 50  0001 C CNN
 F 1 "GND" H 3405 4227 50  0000 C CNN
 F 2 "" H 3400 4400 50  0001 C CNN
@@
 AR Path="/61A047C3/61A2B2C7" Ref="#PWR0205"  Part="1"
 AR Path="/61A55BF3/61A2B2C7" Ref="#PWR0104"  Part="1"
-F 0 "#PWR0104" H 6300 3050 50  0001 C CNN
+F 0 "#PWR0205" H 6300 3050 50  0001 C CNN
 F 1 "+5V" H 6315 3373 50  0000 C CNN
 F 2 "" H 6300 3200 50  0001 C CNN
@@
 AR Path="/61A047C3/61A0A08E" Ref="S201"  Part="1"
 AR Path="/61A55BF3/61A0A08E" Ref="S3001"  Part="1"
-F 0 "S201" H 5450 4260 45  0000 C CNN
+F 0 "S3001" H 5450 4260 45  0000 C CNN
 F 1 "ENCODER-RGB-SWITCH" H 5450 4176 45  0000 C CNN
 F 2 "ENCODER_LED_3" H 5450 4150 20  0001 C CNN
@@
 $EndComp
 $Comp
-L Device:R_Small_US R205
-U 1 1 61A2CA50
-P 6150 3600
-AR Path="/61A047C3/61A2CA50" Ref="R205"  Part="1"
-AR Path="/61A55BF3/61A2CA50" Ref="R3005"  Part="1"
-F 0 "R205" V 5945 3600 50  0000 C CNN
-F 1 "150 5%" V 6036 3600 50  0000 C CNN
-F 2 "Resistor_SMD:R_0805_2012Metric_Pad1.20x1.40mm_HandSolder" H 6150 3600 50  0001 C CNN
-F 3 "https://www.seielect.com/catalog/sei-rmcf_rmcp.pdf" H 6150 3600 50  0001 C CNN
-F 4 "RMCF0805JT150RCT-ND" H 6150 3600 50  0001 C CNN "Digikey PN"
-F 5 "Stackpole Electronics Inc" H 6150 3600 50  0001 C CNN "MFG"
-F 6 "RMCF0805JT150R" H 6150 3600 50  0001 C CNN "MFG #"
-	1    6150 3600
-	0    1    1    0
-$EndComp
-$Comp
-L Device:R_Small_US R208
-U 1 1 61A2D457
-P 7000 3700
-AR Path="/61A047C3/61A2D457" Ref="R208"  Part="1"
-AR Path="/61A55BF3/61A2D457" Ref="R3008"  Part="1"
-F 0 "R208" V 6795 3700 50  0000 C CNN
-F 1 "68 5%" V 6886 3700 50  0000 C CNN
-F 2 "Resistor_SMD:R_0805_2012Metric_Pad1.20x1.40mm_HandSolder" H 7000 3700 50  0001 C CNN
-F 3 "https://www.seielect.com/catalog/sei-rmcf_rmcp.pdf" H 7000 3700 50  0001 C CNN
-F 4 "RMCF0805JT68R0CT-ND" H 7000 3700 50  0001 C CNN "Digikey PN"
-F 5 "Stackpole Electronics Inc" H 7000 3700 50  0001 C CNN "MFG"
-F 6 "RMCF0805JT68R0" H 7000 3700 50  0001 C CNN "MFG #"
-	1    7000 3700
-	0    1    1    0
-$EndComp
-$Comp
-L Device:R_Small_US R209
-U 1 1 61A2DABE
-P 7900 3800
-AR Path="/61A047C3/61A2DABE" Ref="R209"  Part="1"
-AR Path="/61A55BF3/61A2DABE" Ref="R3009"  Part="1"
-F 0 "R209" V 7695 3800 50  0000 C CNN
-F 1 "68 5%" V 7786 3800 50  0000 C CNN
-F 2 "Resistor_SMD:R_0805_2012Metric_Pad1.20x1.40mm_HandSolder" H 7900 3800 50  0001 C CNN
-F 3 "https://www.seielect.com/catalog/sei-rmcf_rmcp.pdf" H 7900 3800 50  0001 C CNN
-F 4 "RMCF0805JT68R0CT-ND" H 7900 3800 50  0001 C CNN "Digikey PN"
-F 5 "Stackpole Electronics Inc" H 7900 3800 50  0001 C CNN "MFG"
-F 6 "RMCF0805JT68R0" H 7900 3800 50  0001 C CNN "MFG #"
-	1    7900 3800
-	0    1    1    0
-$EndComp
-Text HLabel 6250 3600 2    50   Output ~ 0
-REnc_LED_R_5V
-Text HLabel 7100 3700 2    50   Output ~ 0
-REnc_LED_G_5V
-Text HLabel 8000 3800 2    50   Output ~ 0
-REnc_LED_B_5V
-Wire Wire Line
-	6900 3700 6050 3700
-Wire Wire Line
-	6050 3800 7800 3800
-$Comp
 L Device:R_Small_US R206
 U 1 1 61A33A90
@@
 AR Path="/61A047C3/61A33A90" Ref="R206"  Part="1"
 AR Path="/61A55BF3/61A33A90" Ref="R3006"  Part="1"
-F 0 "R206" H 6332 4204 50  0000 R CNN
+F 0 "R3006" H 6332 4204 50  0000 R CNN
 F 1 "2.7k 5%" H 6332 4295 50  0000 R CNN
 F 2 "Resistor_SMD:R_0805_2012Metric_Pad1.20x1.40mm_HandSolder" H 6400 4250 50  0001 C CNN
@@
 AR Path="/61A047C3/61A34096" Ref="R207"  Part="1"
 AR Path="/61A55BF3/61A34096" Ref="R3007"  Part="1"
-F 0 "R207" H 6332 4654 50  0000 R CNN
+F 0 "R3007" H 6332 4654 50  0000 R CNN
 F 1 "4.7k 5%" H 6332 4745 50  0000 R CNN
 F 2 "Resistor_SMD:R_0805_2012Metric_Pad1.20x1.40mm_HandSolder" H 6400 4700 50  0001 C CNN
@@
 AR Path="/61A047C3/61A34367" Ref="C203"  Part="1"
 AR Path="/61A55BF3/61A34367" Ref="C3003"  Part="1"
-F 0 "C203" V 5700 4650 50  0000 L CNN
+F 0 "C3003" V 5700 4650 50  0000 L CNN
 F 1 "1 uF 10% 10V" V 5850 4550 50  0000 L CNN
 F 2 "Capacitor_SMD:C_0805_2012Metric_Pad1.18x1.45mm_HandSolder" H 5950 4700 50  0001 C CNN
@@
 $EndComp
 Wire Wire Line
-	6050 3900 6400 3900
-Wire Wire Line
-	6400 3900 6400 4150
-Wire Wire Line
 	6400 4350 6400 4450
 Wire Wire Line
@@
 AR Path="/61A047C3/61A367C9" Ref="#PWR0204"  Part="1"
 AR Path="/61A55BF3/61A367C9" Ref="#PWR0105"  Part="1"
-F 0 "#PWR0105" H 6200 4950 50  0001 C CNN
+F 0 "#PWR0204" H 6200 4950 50  0001 C CNN
 F 1 "GND" H 6205 5027 50  0000 C CNN
 F 2 "" H 6200 5200 50  0001 C CNN
@@
 Wire Wire Line
 	6200 5100 6200 5200
+Text Label 4300 3400 0    50   ~ 0
+RE_SW_A
+Text Label 4300 3800 0    50   ~ 0
+RE_SW_B
+Text Label 6050 3700 0    50   ~ 0
+RES_DG
+Text Label 6050 3800 0    50   ~ 0
+RES_DB
+Wire Wire Line
+	6400 3900 6400 4150
+Wire Wire Line
+	6050 3900 6400 3900
+Text HLabel 8350 3800 2    50   Output ~ 0
+REnc_LED_B_5V
+Text HLabel 7450 3700 2    50   Output ~ 0
+REnc_LED_G_5V
+Text HLabel 6600 3600 2    50   Output ~ 0
+REnc_LED_R_5V
+$Comp
+L Device:R_Small_US R209
+U 1 1 61A2DABE
+P 8250 3800
+AR Path="/61A047C3/61A2DABE" Ref="R209"  Part="1"
+AR Path="/61A55BF3/61A2DABE" Ref="R3009"  Part="1"
+F 0 "R3009" V 8045 3800 50  0000 C CNN
+F 1 "68 5%" V 8136 3800 50  0000 C CNN
+F 2 "Resistor_SMD:R_0805_2012Metric_Pad1.20x1.40mm_HandSolder" H 8250 3800 50  0001 C CNN
+F 3 "https://www.seielect.com/catalog/sei-rmcf_rmcp.pdf" H 8250 3800 50  0001 C CNN
+F 4 "RMCF0805JT68R0CT-ND" H 8250 3800 50  0001 C CNN "Digikey PN"
+F 5 "Stackpole Electronics Inc" H 8250 3800 50  0001 C CNN "MFG"
+F 6 "RMCF0805JT68R0" H 8250 3800 50  0001 C CNN "MFG #"
+	1    8250 3800
+	0    1    1    0
+$EndComp
+$Comp
+L Device:R_Small_US R208
+U 1 1 61A2D457
+P 7350 3700
+AR Path="/61A047C3/61A2D457" Ref="R208"  Part="1"
+AR Path="/61A55BF3/61A2D457" Ref="R3008"  Part="1"
+F 0 "R3008" V 7145 3700 50  0000 C CNN
+F 1 "68 5%" V 7236 3700 50  0000 C CNN
+F 2 "Resistor_SMD:R_0805_2012Metric_Pad1.20x1.40mm_HandSolder" H 7350 3700 50  0001 C CNN
+F 3 "https://www.seielect.com/catalog/sei-rmcf_rmcp.pdf" H 7350 3700 50  0001 C CNN
+F 4 "RMCF0805JT68R0CT-ND" H 7350 3700 50  0001 C CNN "Digikey PN"
+F 5 "Stackpole Electronics Inc" H 7350 3700 50  0001 C CNN "MFG"
+F 6 "RMCF0805JT68R0" H 7350 3700 50  0001 C CNN "MFG #"
+	1    7350 3700
+	0    1    1    0
+$EndComp
+$Comp
+L Device:R_Small_US R205
+U 1 1 61A2CA50
+P 6500 3600
+AR Path="/61A047C3/61A2CA50" Ref="R205"  Part="1"
+AR Path="/61A55BF3/61A2CA50" Ref="R3005"  Part="1"
+F 0 "R3005" V 6295 3600 50  0000 C CNN
+F 1 "150 5%" V 6386 3600 50  0000 C CNN
+F 2 "Resistor_SMD:R_0805_2012Metric_Pad1.20x1.40mm_HandSolder" H 6500 3600 50  0001 C CNN
+F 3 "https://www.seielect.com/catalog/sei-rmcf_rmcp.pdf" H 6500 3600 50  0001 C CNN
+F 4 "RMCF0805JT150RCT-ND" H 6500 3600 50  0001 C CNN "Digikey PN"
+F 5 "Stackpole Electronics Inc" H 6500 3600 50  0001 C CNN "MFG"
+F 6 "RMCF0805JT150R" H 6500 3600 50  0001 C CNN "MFG #"
+	1    6500 3600
+	0    1    1    0
+$EndComp
+Wire Wire Line
+	6050 3600 6400 3600
+Wire Wire Line
+	6050 3700 7250 3700
+Wire Wire Line
+	6050 3800 8150 3800
+Text Label 6050 3600 0    50   ~ 0
+RES_DR
+Text Label 6050 3900 0    50   ~ 0
+RE_SW_RES
 $EndSCHEMATC

Commit message: Checkpoint
Parts:
- S201: Digikey PN (none) -> 1568-COM-15141-ND; MFG (none) -> SparkFun Electronics; MFG # (none) -> COM-15141; Notes Need from TeachMePCB -> Ordered from Spark Fun directly
Changed lines of the file:
@@
 F 1 "ENCODER-RGB-SWITCH" H 5450 4176 45  0000 C CNN
 F 2 "ENCODER_LED_3" H 5450 4150 20  0001 C CNN
-F 3 "" H 5450 3600 50  0001 C CNN
+F 3 "https://cdn.sparkfun.com/assets/b/8/0/9/9/Part_10997_EC12PLRGBSDVBF-D-25.3K-24-24C-6108-6H__H_.pdf" H 5450 3600 50  0001 C CNN
 F 4 "RES-10859" H 5450 4081 60  0000 C CNN "Field4"
-F 5 "Need from TeachMePCB" H 5450 3600 50  0001 C CNN "Notes"
+F 5 "Ordered from Spark Fun directly" H 5450 3600 50  0001 C CNN "Notes"
+F 6 "1568-COM-15141-ND" H 5450 3600 50  0001 C CNN "Digikey PN"
+F 7 "SparkFun Electronics" H 5450 3600 50  0001 C CNN "MFG"
+F 8 "COM-15141" H 5450 3600 50  0001 C CNN "MFG #"
 	1    5450 3600
 	1    0    0    -1

Commit message: Fix design error in PI4ULS5V201TAEX. Reset and reassigned all annotations.
Parts:
- renumbered C201 to C2901, C202 to C2902, C203 to C2903, R201 to R2901, R202 to R2902, R203 to R2903, R204 to R2904, R206 to R2905, R207 to R2906, R205 to R2907, R208 to R2908, R209 to R2909, S201 to S2901
Changed lines of the file:
@@
 REnc_B
 $Comp
-L power:GND #PWR0203
+L power:GND #PWR02903
 U 1 1 61A23094
 P 4700 3600
-AR Path="/61A047C3/61A23094" Ref="#PWR0203"  Part="1"
-AR Path="/61A55BF3/61A23094" Ref="#PWR0101"  Part="1"
-F 0 "#PWR0203" H 4700 3350 50  0001 C CNN
+AR Path="/61A047C3/61A23094" Ref="#PWR02903"  Part="1"
+AR Path="/61A55BF3/61A23094" Ref="#PWR02803"  Part="1"
+F 0 "#PWR02903" H 4700 3350 50  0001 C CNN
 F 1 "GND" H 4600 3600 50  0000 C CNN
 F 2 "" H 4700 3600 50  0001 C CNN
@@
 	4700 3600 4850 3600
 $Comp
-L power:+3V3 #PWR0202
+L power:+3V3 #PWR02902
 U 1 1 61A247A0
 P 3950 2850
-AR Path="/61A047C3/61A247A0" Ref="#PWR0202"  Part="1"
-AR Path="/61A55BF3/61A247A0" Ref="#PWR0102"  Part="1"
-F 0 "#PWR0202" H 3950 2700 50  0001 C CNN
+AR Path="/61A047C3/61A247A0" Ref="#PWR02902"  Part="1"
+AR Path="/61A55BF3/61A247A0" Ref="#PWR02802"  Part="1"
+F 0 "#PWR02902" H 3950 2700 50  0001 C CNN
 F 1 "+3V3" H 3965 3023 50  0000 C CNN
 F 2 "" H 3950 2850 50  0001 C CNN
@@
 $EndComp
 $Comp
-L Device:R_Small_US R202
+L Device:R_Small_US R2902
 U 1 1 61A24F25
 P 3800 3000
-AR Path="/61A047C3/61A24F25" Ref="R202"  Part="1"
-AR Path="/61A55BF3/61A24F25" Ref="R3002"  Part="1"
-F 0 "R3002" H 4000 2950 50  0000 R CNN
+AR Path="/61A047C3/61A24F25" Ref="R2902"  Part="1"
+AR Path="/61A55BF3/61A24F25" Ref="R2802"  Part="1"
+F 0 "R2902" H 4000 2950 50  0000 R CNN
 F 1 "47k 5%" H 4150 3050 50  0000 R CNN
 F 2 "Resistor_SMD:R_0805_2012Metric_Pad1.20x1.40mm_HandSolder" H 3800 3000 50  0001 C CNN
@@
 $EndComp
 $Comp
-L Device:R_Small_US R204
+L Device:R_Small_US R2904
 U 1 1 61A25788
 P 4100 3000
-AR Path="/61A047C3/61A25788" Ref="R204"  Part="1"
-AR Path="/61A55BF3/61A25788" Ref="R3004"  Part="1"
-F 0 "R3004" H 4032 2954 50  0000 R CNN
+AR Path="/61A047C3/61A25788" Ref="R2904"  Part="1"
+AR Path="/61A55BF3/61A25788" Ref="R2804"  Part="1"
+F 0 "R2904" H 4032 2954 50  0000 R CNN
 F 1 "47k 5%" H 4032 3045 50  0000 R CNN
 F 2 "Resistor_SMD:R_0805_2012Metric_Pad1.20x1.40mm_HandSolder" H 4100 3000 50  0001 C CNN
@@
 Connection ~ 3950 2850
 $Comp
-L Device:R_Small_US R201
+L Device:R_Small_US R2901
 U 1 1 61A260B2
 P 3600 3400
-AR Path="/61A047C3/61A260B2" Ref="R201"  Part="1"
-AR Path="/61A55BF3/61A260B2" Ref="R3001"  Part="1"
-F 0 "R3001" V 3700 3450 50  0000 R CNN
+AR Path="/61A047C3/61A260B2" Ref="R2901"  Part="1"
+AR Path="/61A55BF3/61A260B2" Ref="R2801"  Part="1"
+F 0 "R2901" V 3700 3450 50  0000 R CNN
 F 1 "4.7k 5%" V 3500 3550 50  0000 R CNN
 F 2 "Resistor_SMD:R_0805_2012Metric_Pad1.20x1.40mm_HandSolder" H 3600 3400 50  0001 C CNN
@@
 	3500 3400 3300 3400
 $Comp
-L Device:R_Small_US R203
+L Device:R_Small_US R2903
 U 1 1 61A2753E
 P 3800 3800
-AR Path="/61A047C3/61A2753E" Ref="R203"  Part="1"
-AR Path="/61A55BF3/61A2753E" Ref="R3003"  Part="1"
-F 0 "R3003" V 3900 3850 50  0000 R CNN
+AR Path="/61A047C3/61A2753E" Ref="R2903"  Part="1"
+AR Path="/61A55BF3/61A2753E" Ref="R2803"  Part="1"
+F 0 "R2903" V 3900 3850 50  0000 R CNN
 F 1 "4.7k 5%" V 3700 3950 50  0000 R CNN
 F 2 "Resistor_SMD:R_0805_2012Metric_Pad1.20x1.40mm_HandSolder" H 3800 3800 50  0001 C CNN
@@
 Connection ~ 4100 3800
 $Comp
-L Device:C_Small C201
+L Device:C_Small C2901
 U 1 1 61A2842D
 P 3300 4100
-AR Path="/61A047C3/61A2842D" Ref="C201"  Part="1"
-AR Path="/61A55BF3/61A2842D" Ref="C3001"  Part="1"
-F 0 "C3001" V 3050 4050 50  0000 L CNN
+AR Path="/61A047C3/61A2842D" Ref="C2901"  Part="1"
+AR Path="/61A55BF3/61A2842D" Ref="C2801"  Part="1"
+F 0 "C2901" V 3050 4050 50  0000 L CNN
 F 1 "1 uF 10% 10V" V 3200 3950 50  0000 L CNN
 F 2 "Capacitor_SMD:C_0805_2012Metric_Pad1.18x1.45mm_HandSolder" H 3300 4100 50  0001 C CNN
@@
 $EndComp
 $Comp
-L Device:C_Small C202
+L Device:C_Small C2902
 U 1 1 61A29140
 P 3500 4100
-AR Path="/61A047C3/61A29140" Ref="C202"  Part="1"
-AR Path="/61A55BF3/61A29140" Ref="C3002"  Part="1"
-F 0 "C3002" V 3250 4050 50  0000 L CNN
+AR Path="/61A047C3/61A29140" Ref="C2902"  Part="1"
+AR Path="/61A55BF3/61A29140" Ref="C2802"  Part="1"
+F 0 "C2902" V 3250 4050 50  0000 L CNN
 F 1 "1 uF 10% 10V" V 3400 3950 50  0000 L CNN
 F 2 "Capacitor_SMD:C_0805_2012Metric_Pad1.18x1.45mm_HandSolder" H 3500 4100 50  0001 C CNN
@@
 Connection ~ 3500 3800
 $Comp
-L power:GND #PWR0201
+L power:GND #PWR02901
 U 1 1 61A2A062
 P 3400 4400
-AR Path="/61A047C3/61A2A062" Ref="#PWR0201"  Part="1"
-AR Path="/61A55BF3/61A2A062" Ref="#PWR0103"  Part="1"
-F 0 "#PWR0201" H 3400 4150 50  0001 C CNN
+AR Path="/61A047C3/61A2A062" Ref="#PWR02901"  Part="1"
+AR Path="/61A55BF3/61A2A062" Ref="#PWR02801"  Part="1"
+F 0 "#PWR02901" H 3400 4150 50  0001 C CNN
 F 1 "GND" H 3405 4227 50  0000 C CNN
 F 2 "" H 3400 4400 50  0001 C CNN
@@
 Connection ~ 3400 4200
 $Comp
-L power:+5V #PWR0205
+L power:+5V #PWR02905
 U 1 1 61A2B2C7
 P 6300 3200
-AR Path="/61A047C3/61A2B2C7" Ref="#PWR0205"  Part="1"
-AR Path="/61A55BF3/61A2B2C7" Ref="#PWR0104"  Part="1"
-F 0 "#PWR0205" H 6300 3050 50  0001 C CNN
+AR Path="/61A047C3/61A2B2C7" Ref="#PWR02905"  Part="1"
+AR Path="/61A55BF3/61A2B2C7" Ref="#PWR02805"  Part="1"
+F 0 "#PWR02905" H 6300 3050 50  0001 C CNN
 F 1 "+5V" H 6315 3373 50  0000 C CNN
 F 2 "" H 6300 3200 50  0001 C CNN
@@
 	6300 3300 6050 3300
 $Comp
-L TMPCB_R2:ENCODER-RGB-SWITCH S201
+L TMPCB_R2:ENCODER-RGB-SWITCH S2901
 U 1 1 61A0A08E
 P 5450 3600
-AR Path="/61A047C3/61A0A08E" Ref="S201"  Part="1"
-AR Path="/61A55BF3/61A0A08E" Ref="S3001"  Part="1"
-F 0 "S3001" H 5450 4260 45  0000 C CNN
+AR Path="/61A047C3/61A0A08E" Ref="S2901"  Part="1"
+AR Path="/61A55BF3/61A0A08E" Ref="S2801"  Part="1"
+F 0 "S2901" H 5450 4260 45  0000 C CNN
 F 1 "ENCODER-RGB-SWITCH" H 5450 4176 45  0000 C CNN
 F 2 "ENCODER_LED_3" H 5450 4150 20  0001 C CNN
@@
 $EndComp
 $Comp
-L Device:R_Small_US R206
+L Device:R_Small_US R2905
 U 1 1 61A33A90
 P 6400 4250
-AR Path="/61A047C3/61A33A90" Ref="R206"  Part="1"
-AR Path="/61A55BF3/61A33A90" Ref="R3006"  Part="1"
-F 0 "R3006" H 6332 4204 50  0000 R CNN
+AR Path="/61A047C3/61A33A90" Ref="R2905"  Part="1"
+AR Path="/61A55BF3/61A33A90" Ref="R2805"  Part="1"
+F 0 "R2905" H 6332 4204 50  0000 R CNN
 F 1 "2.7k 5%" H 6332 4295 50  0000 R CNN
 F 2 "Resistor_SMD:R_0805_2012Metric_Pad1.20x1.40mm_HandSolder" H 6400 4250 50  0001 C CNN
@@
 $EndComp
 $Comp
-L Device:R_Small_US R207
+L Device:R_Small_US R2906
 U 1 1 61A34096
 P 6400 4700
-AR Path="/61A047C3/61A34096" Ref="R207"  Part="1"
-AR Path="/61A55BF3/61A34096" Ref="R3007"  Part="1"
-F 0 "R3007" H 6332 4654 50  0000 R CNN
+AR Path="/61A047C3/61A34096" Ref="R2906"  Part="1"
+AR Path="/61A55BF3/61A34096" Ref="R2806"  Part="1"
+F 0 "R2906" H 6332 4654 50  0000 R CNN
 F 1 "4.7k 5%" H 6332 4745 50  0000 R CNN
 F 2 "Resistor_SMD:R_0805_2012Metric_Pad1.20x1.40mm_HandSolder" H 6400 4700 50  0001 C CNN
@@
 $EndComp
 $Comp
-L Device:C_Small C203
+L Device:C_Small C2903
 U 1 1 61A34367
 P 5950 4700
-AR Path="/61A047C3/61A34367" Ref="C203"  Part="1"
-AR Path="/61A55BF3/61A34367" Ref="C3003"  Part="1"
-F 0 "C3003" V 5700 4650 50  0000 L CNN
+AR Path="/61A047C3/61A34367" Ref="C2903"  Part="1"
+AR Path="/61A55BF3/61A34367" Ref="C2803"  Part="1"
+F 0 "C2903" V 5700 4650 50  0000 L CNN
 F 1 "1 uF 10% 10V" V 5850 4550 50  0000 L CNN
 F 2 "Capacitor_SMD:C_0805_2012Metric_Pad1.18x1.45mm_HandSolder" H 5950 4700 50  0001 C CNN
@@
 	5950 5100 6200 5100
 $Comp
-L power:GND #PWR0204
+L power:GND #PWR02904
 U 1 1 61A367C9
 P 6200 5200
-AR Path="/61A047C3/61A367C9" Ref="#PWR0204"  Part="1"
-AR Path="/61A55BF3/61A367C9" Ref="#PWR0105"  Part="1"
-F 0 "#PWR0204" H 6200 4950 50  0001 C CNN
+AR Path="/61A047C3/61A367C9" Ref="#PWR02904"  Part="1"
+AR Path="/61A55BF3/61A367C9" Ref="#PWR02804"  Part="1"
+F 0 "#PWR02904" H 6200 4950 50  0001 C CNN
 F 1 "GND" H 6205 5027 50  0000 C CNN
 F 2 "" H 6200 5200 50  0001 C CNN
@@
 REnc_LED_R_5V
 $Comp
-L Device:R_Small_US R209
+L Device:R_Small_US R2909
 U 1 1 61A2DABE
 P 8250 3800
-AR Path="/61A047C3/61A2DABE" Ref="R209"  Part="1"
-AR Path="/61A55BF3/61A2DABE" Ref="R3009"  Part="1"
-F 0 "R3009" V 8045 3800 50  0000 C CNN
+AR Path="/61A047C3/61A2DABE" Ref="R2909"  Part="1"
+AR Path="/61A55BF3/61A2DABE" Ref="R2809"  Part="1"
+F 0 "R2909" V 8045 3800 50  0000 C CNN
 F 1 "68 5%" V 8136 3800 50  0000 C CNN
 F 2 "Resistor_SMD:R_0805_2012Metric_Pad1.20x1.40mm_HandSolder" H 8250 3800 50  0001 C CNN
@@
 $EndComp
 $Comp
-L Device:R_Small_US R208
+L Device:R_Small_US R2908
 U 1 1 61A2D457
 P 7350 3700
-AR Path="/61A047C3/61A2D457" Ref="R208"  Part="1"
-AR Path="/61A55BF3/61A2D457" Ref="R3008"  Part="1"
-F 0 "R3008" V 7145 3700 50  0000 C CNN
+AR Path="/61A047C3/61A2D457" Ref="R2908"  Part="1"
+AR Path="/61A55BF3/61A2D457" Ref="R2808"  Part="1"
+F 0 "R2908" V 7145 3700 50  0000 C CNN
 F 1 "68 5%" V 7236 3700 50  0000 C CNN
 F 2 "Resistor_SMD:R_0805_2012Metric_Pad1.20x1.40mm_HandSolder" H 7350 3700 50  0001 C CNN
@@
 $EndComp
 $Comp
-L Device:R_Small_US R205
+L Device:R_Small_US R2907
 U 1 1 61A2CA50
 P 6500 3600
-AR Path="/61A047C3/61A2CA50" Ref="R205"  Part="1"
-AR Path="/61A55BF3/61A2CA50" Ref="R3005"  Part="1"
-F 0 "R3005" V 6295 3600 50  0000 C CNN
+AR Path="/61A047C3/61A2CA50" Ref="R2907"  Part="1"
+AR Path="/61A55BF3/61A2CA50" Ref="R2807"  Part="1"
+F 0 "R2907" V 6295 3600 50  0000 C CNN
 F 1 "150 5%" V 6386 3600 50  0000 C CNN
 F 2 "Resistor_SMD:R_0805_2012Metric_Pad1.20x1.40mm_HandSolder" H 6500 3600 50  0001 C CNN
