File: RotaryEncoder.sch (KiCad schematic (older format))
At the start: 13 parts

Commit message: Updated Switch to use Bournes P/N PEL12T-4225S-S1024, Update Connector to use Amphenol F31L-1A7H1-11024
Parts:
- S2901: Digikey PN 1568-COM-15141-ND -> PEL12T-4225S-S1024-ND; MFG SparkFun Electronics -> Bournes; MFG # COM-15141 -> PEL12T-4225S-S1024; Notes Ordered from Spark Fun directly -> (none)
Changed lines of the file:
@@
 F 3 "https://cdn.sparkfun.com/assets/b/8/0/9/9/Part_10997_EC12PLRGBSDVBF-D-25.3K-24-24C-6108-6H__H_.pdf" H 5450 3600 50  0001 C CNN
 F 4 "RES-10859" H 5450 4081 60  0000 C CNN "Field4"
-F 5 "Ordered from Spark Fun directly" H 5450 3600 50  0001 C CNN "Notes"
-F 6 "1568-COM-15141-ND" H 5450 3600 50  0001 C CNN "Digikey PN"
-F 7 "SparkFun Electronics" H 5450 3600 50  0001 C CNN "MFG"
-F 8 "COM-15141" H 5450 3600 50  0001 C CNN "MFG #"
+F 5 "" H 5450 3600 50  0001 C CNN "Notes"
+F 6 "PEL12T-4225S-S1024-ND" H 5450 3600 50  0001 C CNN "Digikey PN"
+F 7 "Bournes" H 5450 3600 50  0001 C CNN "MFG"
+F 8 "PEL12T-4225S-S1024" H 5450 3600 50  0001 C CNN "MFG #"
 	1    5450 3600
 	1    0    0    -1
