File: eInkDisplay.sch (KiCad schematic (older format))
At the start: 16 parts, among them J2701 FPC 1x24, Q2701 Q_PJFET_GDS

Commit message: Updated Switch to use Bournes P/N PEL12T-4225S-S1024, Update Connector to use Amphenol F31L-1A7H1-11024
Parts:
- J2701: Digikey PN WM20872CT-ND -> 609-F31L-1A7H1-11024CT-ND; MFG Molex -> Amphenol ICC (FCI); MFG # 5052782433 -> F31L-1A7H1-11024
Changed lines of the file:
@@
 F 2 "Macro Keyboard:Amphenol_F31L-1A7H1-11024" H 8000 3750 50  0001 C CNN
 F 3 "https://www.molex.com/pdm_docs/sd/5052782433_sd.pdf" H 8000 3750 50  0001 C CNN
-F 4 "WM20872CT-ND" H 8000 3750 50  0001 C CNN "Digikey PN"
-F 5 "Molex" H 8000 3750 50  0001 C CNN "MFG"
-F 6 "5052782433" H 8000 3750 50  0001 C CNN "MFG #"
+F 4 "609-F31L-1A7H1-11024CT-ND" H 8000 3750 50  0001 C CNN "Digikey PN"
+F 5 "Amphenol ICC (FCI)" H 8000 3750 50  0001 C CNN "MFG"
+F 6 "F31L-1A7H1-11024" H 8000 3750 50  0001 C CNN "MFG #"
 	1    8000 3750
 	1    0    0    -1
