File: Macro Keyboard.sch (KiCad schematic (older format))
At the start: 0 parts

Commit message: Use GP25_LED for ePaper RESET
Note: This replaces R6/196a722 in its entirety.

IS: J2901 (Connector for epaper) Pin 10 (Reset) connected to +3.3V via R2902 (100k ohm)
SHOULD BE: J2901 Pin 10 connected to U2801 Pin 48 (GPIO25_LED aka TP5)
Changed lines of the file:
@@
-$EndSheet
-$Sheet
-S 2450 2150 550  1100
-U 61A0B595
-F0 "10 Group Switch" 50
-F1 "10GroupSwitch.sch" 50
-F2 "SW01" O R 3000 2200 50
-F3 "SW02" O R 3000 2350 50
-F4 "SW03" O R 3000 2850 50
-F5 "SW04" O R 3000 3150 50
-F6 "SW05" O R 3000 3050 50
-F7 "SW06" O R 3000 2750 50
-F8 "SW07" O R 3000 2450 50
-F9 "SW08" O R 3000 2550 50
-F10 "SW09" O R 3000 2650 50
-F11 "SW10" O R 3000 2950 50
 $EndSheet
 $Sheet
@@
 Wire Wire Line
 	3550 3050 3000 3050
-Wire Wire Line
-	3000 3150 3350 3150
 $Sheet
 S 6650 2700 800  500
@@
 F26 "GPIO_27_ADC1" B L 3550 3500 50
 F27 "GPIO_28_ADC2" B L 3550 3400 50
-$EndSheet
-Wire Wire Line
-	6650 2750 5700 2750
-Wire Wire Line
-	5700 2750 5700 1800
-Wire Wire Line
-	5700 1800 2350 1800
-Wire Wire Line
-	2350 1800 2350 3200
-Wire Wire Line
-	2350 3200 3350 3200
-Wire Wire Line
-	3350 3200 3350 3150
-Connection ~ 3350 3150
-Wire Wire Line
-	3350 3150 3550 3150
+F28 "GPIO25_LED" I R 5250 2300 50
+$EndSheet
+$Sheet
+S 2450 2150 550  1100
+U 61A0B595
+F0 "10 Group Switch" 50
+F1 "10GroupSwitch.sch" 50
+F2 "SW01" O R 3000 2200 50
+F3 "SW02" O R 3000 2350 50
+F4 "SW03" O R 3000 2850 50
+F5 "SW04" O R 3000 3150 50
+F6 "SW05" O R 3000 3050 50
+F7 "SW06" O R 3000 2750 50
+F8 "SW07" O R 3000 2450 50
+F9 "SW08" O R 3000 2550 50
+F10 "SW09" O R 3000 2650 50
+F11 "SW10" O R 3000 2950 50
+$EndSheet
+Wire Wire Line
+	3000 3150 3550 3150
+Wire Wire Line
+	6650 2750 5850 2750
+Wire Wire Line
+	5850 2750 5850 2300
+Wire Wire Line
+	5850 2300 5250 2300
 $EndSCHEMATC
